File: centered_diodes/tin52holyiot.kicad_pcb (KiCad board)
At the start: 2 copper layers, 285 x 94.6 mm, 165 parts

Commit message: added mx version and some variations, new power switch
Parts:
- removed the REF** at (76.1, 17.8)
- removed the REF** at (218.9, 17.8)
- added REF**: RollerEncoder_Panasonic_EVQWGD001, RollerEncoder_Panasonic_EVQWGD001, F.Cu at (74.6, 23.4)
- added REF**: RollerEncoder_Panasonic_EVQWGD001, RollerEncoder_Panasonic_EVQWGD001, F.Cu at (215.8, 23.4)
- moved S87 8.75 mm to (192.7, -7.45)
- moved S88 8.75 mm to (192.7, -7.45)
- moved S91 8.75 mm to (185.0, -36.4)
- moved S92 8.75 mm to (185.0, -36.4)
- moved S89 8.75 mm to (188.8, -21.9)
- moved S90 8.75 mm to (188.8, -21.9)
- moved S100 8.75 mm to (167.5, -30.0)
- moved S99 8.75 mm to (167.5, -30.0)
- moved ? 8.75 mm to (145.2, -37.0)
- moved JST1 8.75 mm to (152.8, -18.6)
- moved S33 8.75 mm to (93.9, 7.04)
- moved S34 8.75 mm to (93.9, 7.04)
- moved T1 8.75 mm to (137.6, -18.6)
- moved S47 8.75 mm to (122.9, -30.0)
- moved S48 8.75 mm to (122.9, -30.0)
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Other:
- board size 285 x 94.6 mm -> 285 x 97.2 mm
